File: E_Rudziks_MultiVib/E_Rudziks_MultiVib.sch (KiCad schematic (older format))
At the start: 11 parts

Commit message: Update E_Rudziks_MultiVib.sch
Parts:
- removed Q? (x2): BC548, TO-92, symbol Transistor_BJT:BC548
- added U1: LTC4300-1, symbol Buffer:LTC4300-1
- gave numbers to parts that had none: 9
Connections:
- net at BT1.1 (+), D1.2 (A), D2.2 (A)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: now also C1.1, C2.1, U1.1 (VCC2), U1.5 (ACC), U1.8 (VCC)
- net at R4.2: now also U1.7 (SDAOUT); no longer C2.1
- net at R3.2: now also U1.2 (SCLOUT); no longer C2.2
- net at R2.2: now also U1.6 (SDAIN); no longer C1.2
- net at R1.2: now also U1.3 (SCLIN); no longer C1.1
- net at BT1.2 (-): now also U1.4 (GND)
- new net GND: C1.2, C2.2
Other:
- moved on the sheet: C1, C2
Changed lines of the file:
@@
 $EndDescr
 $Comp
-L Device:LED D?
+L Device:LED D2
 U 1 1 5F93EAB2
 P 7450 2700
-F 0 "D?" V 7489 2582 50  0000 R CNN
+F 0 "D2" V 7489 2582 50  0000 R CNN
 F 1 "LED" V 7398 2582 50  0000 R CNN
 F 2 "" H 7450 2700 50  0001 C CNN
@@
 $EndComp
 $Comp
-L Device:LED D?
+L Device:LED D1
 U 1 1 5F93EF93
 P 5750 2700
-F 0 "D?" V 5789 2582 50  0000 R CNN
+F 0 "D1" V 5789 2582 50  0000 R CNN
 F 1 "LED" V 5698 2582 50  0000 R CNN
 F 2 "" H 5750 2700 50  0001 C CNN
@@
 $EndComp
 $Comp
-L Device:R R?
+L Device:R R4
 U 1 1 5F93FA00
 P 7450 3150
-F 0 "R?" H 7520 3196 50  0000 L CNN
+F 0 "R4" H 7520 3196 50  0000 L CNN
 F 1 "470R" H 7520 3105 50  0000 L CNN
 F 2 "" V 7380 3150 50  0001 C CNN
@@
 $EndComp
 $Comp
-L Device:R R?
+L Device:R R3
 U 1 1 5F93FEE5
 P 6900 3150
-F 0 "R?" H 6970 3196 50  0000 L CNN
+F 0 "R3" H 6970 3196 50  0000 L CNN
 F 1 "47K" H 6970 3105 50  0000 L CNN
 F 2 "" V 6830 3150 50  0001 C CNN
@@
 $EndComp
 $Comp
-L Device:R R?
+L Device:R R2
 U 1 1 5F940499
 P 6300 3150
-F 0 "R?" H 6370 3196 50  0000 L CNN
+F 0 "R2" H 6370 3196 50  0000 L CNN
 F 1 "47K" H 6370 3105 50  0000 L CNN
 F 2 "" V 6230 3150 50  0001 C CNN
@@
 $EndComp
 $Comp
-L Device:R R?
+L Device:R R1
 U 1 1 5F94098E
 P 5750 3150
-F 0 "R?" H 5820 3196 50  0000 L CNN
+F 0 "R1" H 5820 3196 50  0000 L CNN
 F 1 "470R" H 5820 3105 50  0000 L CNN
 F 2 "" V 5680 3150 50  0001 C CNN
@@
 $EndComp
 $Comp
-L Device:CP C?
+L Device:CP C1
 U 1 1 5F941812
-P 6050 3500
-F 0 "C?" V 6305 3500 50  0000 C CNN
-F 1 "47uF" V 6214 3500 50  0000 C CNN
-F 2 "" H 6088 3350 50  0001 C CNN
-F 3 "~" H 6050 3500 50  0001 C CNN
-	1    6050 3500
-	0    -1   -1   0
-$EndComp
-$Comp
-L Device:CP C?
+P 6200 2750
+F 0 "C1" V 6455 2750 50  0000 C CNN
+F 1 "47uF" V 6364 2750 50  0000 C CNN
+F 2 "" H 6238 2600 50  0001 C CNN
+F 3 "~" H 6200 2750 50  0001 C CNN
+	1    6200 2750
+	1    0    0    -1
+$EndComp
+$Comp
+L Device:CP C2
 U 1 1 5F941F76
-P 7250 3500
-F 0 "C?" V 6995 3500 50  0000 C CNN
-F 1 "47uF" V 7086 3500 50  0000 C CNN
-F 2 "" H 7288 3350 50  0001 C CNN
-F 3 "~" H 7250 3500 50  0001 C CNN
-	1    7250 3500
-	0    1    1    0
-$EndComp
-Wire Wire Line
-	5900 3500 5750 3500
-Wire Wire Line
-	5750 3500 5750 3300
+P 7250 2950
+F 0 "C2" V 6995 2950 50  0000 C CNN
+F 1 "47uF" V 7086 2950 50  0000 C CNN
+F 2 "" H 7288 2800 50  0001 C CNN
+F 3 "~" H 7250 2950 50  0001 C CNN
+	1    7250 2950
+	1    0    0    -1
+$EndComp
 Wire Wire Line
 	5750 3000 5750 2850
 Wire Wire Line
 	5750 2550 5750 2500
-Wire Wire Line
-	5750 2500 6300 2500
 Wire Wire Line
 	7450 2500 7450 2550
@@
 Connection ~ 6900 2500
 Wire Wire Line
-	6900 2500 7450 2500
+	6900 2500 7250 2500
 Wire Wire Line
 	6300 3000 6300 2500
 Connection ~ 6300 2500
 Wire Wire Line
-	6300 2500 6900 2500
+	6300 2500 6550 2500
 Wire Wire Line
 	7450 2850 7450 3000
-Wire Wire Line
-	7450 3300 7450 3500
-Wire Wire Line
-	7450 3500 7400 3500
-Wire Wire Line
-	7100 3500 6900 3500
-Wire Wire Line
-	6900 3500 6900 3300
-Wire Wire Line
-	6200 3500 6300 3500
-Wire Wire Line
-	6300 3500 6300 3300
-$Comp
-L Transistor_BJT:BC548 Q?
-U 1 1 5F9433C6
-P 7350 4000
-F 0 "Q?" H 7540 4091 50  0000 L CNN
-F 1 "BC548" H 7540 4000 50  0000 L CNN
-F 2 "TO-92" H 7540 3909 50  0000 L CIN
-F 3 "http://www.fairchildsemi.com/ds/BC/BC547.pdf" H 7350 4000 50  0001 L CNN
-	1    7350 4000
-	1    0    0    -1
-$EndComp
-$Comp
-L Transistor_BJT:BC548 Q?
-U 1 1 5F94455C
-P 5850 4000
-F 0 "Q?" H 6041 3909 50  0000 L CNN
-F 1 "BC548" H 6041 4000 50  0000 L CNN
-F 2 "TO-92" H 6041 4091 50  0000 L CIN
-F 3 "http://www.fairchildsemi.com/ds/BC/BC547.pdf" H 5850 4000 50  0001 L CNN
-	1    5850 4000
-	-1   0    0    1
-$EndComp
-Wire Wire Line
-	5750 3500 5750 3800
-Connection ~ 5750 3500
-Wire Wire Line
-	7450 3500 7450 3800
-Connection ~ 7450 3500
-Wire Wire Line
-	6050 4000 6900 4000
-Wire Wire Line
-	6900 4000 6900 3500
-Connection ~ 6900 3500
-Wire Wire Line
-	7150 4000 7000 4000
-Wire Wire Line
-	7000 4000 7000 3900
-Wire Wire Line
-	7000 3900 6300 3900
-Wire Wire Line
-	6300 3900 6300 3500
-Connection ~ 6300 3500
-Wire Wire Line
-	7450 4200 7450 4500
-Wire Wire Line
-	7450 4500 5750 4500
-Wire Wire Line
-	5750 4500 5750 4200
-$Comp
-L Device:Battery BT?
+$Comp
+L Device:Battery BT1
 U 1 1 5F946B12
 P 5200 3500
-F 0 "BT?" H 5308 3546 50  0000 L CNN
+F 0 "BT1" H 5308 3546 50  0000 L CNN
 F 1 "9V" H 5308 3455 50  0000 L CNN
 F 2 "" V 5200 3560 50  0001 C CNN
@@
 	5200 3700 5200 4500
 Wire Wire Line
-	5200 4500 5750 4500
-Connection ~ 5750 4500
-Wire Wire Line
 	5200 3300 5200 2500
 Wire Wire Line
 	5200 2500 5750 2500
 Connection ~ 5750 2500
+$Comp
+L Buffer:LTC4300-1 U1
+U 1 1 5F95E639
+P 6600 3500
+F 0 "U1" H 6600 3625 50  0000 C CNN
+F 1 "LTC4300-1" H 6600 3534 50  0000 C CNN
+F 2 "" H 6600 3500 50  0001 C CNN
+F 3 "" H 6600 3500 50  0001 C CNN
+	1    6600 3500
+	1    0    0    -1
+$EndComp
+Wire Wire Line
+	6150 3600 6150 3400
+Wire Wire Line
+	6150 3400 6550 3400
+Wire Wire Line
+	6550 3400 6550 2500
+Connection ~ 6550 2500
+Wire Wire Line
+	6550 2500 6650 2500
+Wire Wire Line
+	7050 3600 7050 3400
+Wire Wire Line
+	7050 3400 6650 3400
+Wire Wire Line
+	6650 3400 6650 2500
+Connection ~ 6650 2500
+Wire Wire Line
+	6650 2500 6900 2500
+Wire Wire Line
+	7250 2800 7250 2500
+Connection ~ 7250 2500
+Wire Wire Line
+	7250 2500 7450 2500
+Wire Wire Line
+	6150 3900 6150 4500
+Wire Wire Line
+	6150 3800 5750 3800
+Wire Wire Line
+	5750 3300 5750 3800
+Wire Wire Line
+	7050 3800 7200 3800
+Wire Wire Line
+	7200 3800 7200 4000
+Wire Wire Line
+	7200 4000 6050 4000
+Wire Wire Line
+	6050 4000 6050 3300
+Wire Wire Line
+	6050 3300 6300 3300
+Wire Wire Line
+	6150 3700 6100 3700
+Wire Wire Line
+	6100 3700 6100 3350
+Wire Wire Line
+	6100 3350 6500 3350
+Wire Wire Line
+	6500 3350 6500 3300
+Wire Wire Line
+	6500 3300 6900 3300
+Wire Wire Line
+	7050 3700 7450 3700
+Wire Wire Line
+	7450 3300 7450 3700
+Wire Wire Line
+	7050 3900 7800 3900
+Wire Wire Line
+	7800 3900 7800 2500
+Wire Wire Line
+	7800 2500 7450 2500
+Connection ~ 7450 2500
+Wire Wire Line
+	5200 4500 6150 4500
+$Comp
+L power:GND #PWR01
+U 1 1 5F96893E
+P 6200 2900
+F 0 "#PWR01" H 6200 2650 50  0001 C CNN
+F 1 "GND" H 6205 2727 50  0000 C CNN
+F 2 "" H 6200 2900 50  0001 C CNN
+F 3 "" H 6200 2900 50  0001 C CNN
+	1    6200 2900
+	1    0    0    -1
+$EndComp
+Wire Wire Line
+	5750 2500 6200 2500
+Wire Wire Line
+	6200 2600 6200 2500
+Connection ~ 6200 2500
+Wire Wire Line
+	6200 2500 6300 2500
+$Comp
+L power:GND #PWR02
+U 1 1 5F96A49A
+P 7250 3100
+F 0 "#PWR02" H 7250 2850 50  0001 C CNN
+F 1 "GND" H 7255 2927 50  0000 C CNN
+F 2 "" H 7250 3100 50  0001 C CNN
+F 3 "" H 7250 3100 50  0001 C CNN
+	1    7250 3100
+	1    0    0    -1
+$EndComp
 $EndSCHEMATC
